Commit message: update 3D lidar

File: ugv_ws/src/ugv_description/urdf/ugv.gazebo.xacro (robot description, xacro)
@@ -68,4 +68,45 @@
     </sensor>
   </gazebo>
+    <!-- ===================== 3D LIDAR (multi-channel point cloud) ===================== -->
+  <gazebo reference="lidar_3d_link">
+    <sensor name="lidar_3d" type="ray">
+      <pose>0 0 0 0 0 0</pose>
+      <visualize>false</visualize>
+      <update_rate>5</update_rate>
+      <ray>
+        <scan>
+          <horizontal>
+            <samples>180</samples>
+            <resolution>1</resolution>
+            <min_angle>-3.14159</min_angle>
+            <max_angle>3.14159</max_angle>
+          </horizontal>
+          <vertical>
+            <samples>8</samples>
+            <resolution>1</resolution>
+            <min_angle>-0.2618</min_angle>
+            <max_angle>0.2618</max_angle>
+          </vertical>
+        </scan>
+        <range>
+          <min>0.3</min>
+          <max>15.0</max>
+          <resolution>0.03</resolution>
+        </range>
+        <noise>
+          <type>gaussian</type>
+          <mean>0.0</mean>
+          <stddev>0.02</stddev>
+        </noise>
+      </ray>
+      <plugin name="lidar_3d_plugin" filename="libgazebo_ros_ray_sensor.so">
+        <ros>
+          <remapping>~/out:=points</remapping>
+        </ros>
+        <output_type>sensor_msgs/PointCloud2</output_type>
+        <frame_name>lidar_3d_link</frame_name>
+      </plugin>
+    </sensor>
+  </gazebo>
   <!-- ===================== IMU ===================== -->
   <gazebo reference="imu_link">

File: ugv_ws/src/ugv_description/urdf/ugv.urdf.xacro (robot description, xacro)
@@ -98,4 +98,23 @@
     <origin xyz="0.15 0 ${base_height/2 + 0.03}" rpy="0 0 0"/>
   </joint>
+    <!-- ===================== 3D LIDAR ===================== -->
+  <link name="lidar_3d_link">
+    <visual>
+      <geometry><cylinder radius="0.05" length="0.08"/></geometry>
+      <material name="black"/>
+    </visual>
+    <collision>
+      <geometry><cylinder radius="0.05" length="0.08"/></geometry>
+    </collision>
+    <inertial>
+      <mass value="0.3"/>
+      <inertia ixx="0.0002" ixy="0" ixz="0" iyy="0.0002" iyz="0" izz="0.0002"/>
+    </inertial>
+  </link>
+  <joint name="lidar_3d_joint" type="fixed">
+    <parent link="base_link"/>
+    <child link="lidar_3d_link"/>
+    <origin xyz="0.10 0 ${base_height/2 + 0.10}" rpy="0 0 0"/>
+  </joint>
   <!-- ===================== IMU ===================== -->
   <link name="imu_link">
